File: circuit/macroglider/macroglider.kicad_sch (KiCad schematic)
At the start: 46 parts, among them SW1 Capacitive Button, SW2 Capacitive Button, SW3 Capacitive Button, SW4 Capacitive Button, SW5 Capacitive Button, SW6 Capacitive Button, SW7 Capacitive Button, SW8 Capacitive Button, SW9 Capacitive Button, U1 Pico

Commit message: changes
Parts:
- OLED1: footprint easyeda2kicad:OLED-TH_L35.4-W33.5_HS13L03W2C01 -> easyeda2kicad:OLED-TH_L35.4-W33.5_HS13L03W2C01_without_mount_outline
Connections:
- net FADER1B: now also U1.7 (GPIO5); no longer U1.1 (GPIO0)
- net FADER1C: now also U1.31 (GPIO26_ADC0); no longer U1.34 (GPIO28_ADC2)
- net FADER2A: now also U1.4 (GPIO2); no longer U1.7 (GPIO5)
- net FADER2B: now also U1.5 (GPIO3); no longer U1.2 (GPIO1)
- net FADER3A: now also U1.1 (GPIO0); no longer U1.5 (GPIO3)
- net FADER3B: now also U1.2 (GPIO1); no longer U1.4 (GPIO2)
- net FADER3C: now also U1.34 (GPIO28_ADC2); no longer U1.31 (GPIO26_ADC0)
- net ROT1A: now also U1.11 (GPIO8); no longer U1.10 (GPIO7)
- net ROT1B: now also U1.9 (GPIO6); no longer U1.11 (GPIO8)
- net ROT1C: now also U1.10 (GPIO7); no longer U1.12 (GPIO9)
- net ROT2A: now also U1.12 (GPIO9); no longer U1.14 (GPIO10)
- net ROT2C: now also U1.14 (GPIO10); no longer U1.16 (GPIO12)
- net TPAD8: now also U1.16 (GPIO12); no longer U1.9 (GPIO6)
Changed lines of the file:
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@@
 		)
 	)
-	(label "FADER3B"
+	(label "FADER2A"
 		(at 22.86 41.91 0)
 		(fields_autoplaced yes)
@@
 		)
 	)
-	(label "FADER1B"
+	(label "FADER3A"
 		(at 22.86 34.29 0)
 		(fields_autoplaced yes)
@@
 		)
 	)
-	(label "ROT1A"
+	(label "ROT1C"
 		(at 22.86 57.15 0)
 		(fields_autoplaced yes)
@@
 		)
 	)
-	(label "FADER2B"
+	(label "FADER3B"
 		(at 22.86 36.83 0)
 		(fields_autoplaced yes)
@@
 		)
 	)
-	(label "ROT1C"
+	(label "ROT2A"
 		(at 22.86 62.23 0)
 		(fields_autoplaced yes)
@@
 		)
 	)
-	(label "TPAD8"
+	(label "ROT1B"
 		(at 22.86 54.61 0)
 		(fields_autoplaced yes)
@@
 		)
 	)
-	(label "ROT1B"
+	(label "ROT1A"
 		(at 22.86 59.69 0)
 		(fields_autoplaced yes)
@@
 		)
 	)
-	(label "ROT2A"
+	(label "ROT2C"
 		(at 22.86 67.31 0)
 		(fields_autoplaced yes)
@@
 		)
 	)
-	(label "FADER1C"
+	(label "FADER3C"
 		(at 76.2 49.53 0)
 		(fields_autoplaced yes)
@@
 		)
 	)
-	(label "FADER2A"
+	(label "FADER1B"
 		(at 22.86 49.53 0)
 		(fields_autoplaced yes)
@@
 		)
 	)
-	(label "ROT2C"
+	(label "TPAD8"
 		(at 22.86 72.39 0)
 		(fields_autoplaced yes)
@@
 		)
 	)
-	(label "FADER3C"
+	(label "FADER1C"
 		(at 76.2 57.15 0)
 		(fields_autoplaced yes)
@@
 		)
 	)
-	(label "FADER3A"
+	(label "FADER2B"
 		(at 22.86 44.45 0)
 		(fields_autoplaced yes)
@@
 			)
 		)
-		(property "Footprint" "easyeda2kicad:OLED-TH_L35.4-W33.5_HS13L03W2C01"
+		(property "Footprint" "easyeda2kicad:OLED-TH_L35.4-W33.5_HS13L03W2C01_without_mount_outline"
 			(at 93.98 120.65 0)
 			(effects
